Commit message: Update 3dof geometry
Update 3dof to reflect geometry of robot

File: urdf/threeDOF.urdf (robot description, URDF)
Before this commit: robot threeDOF, 16 links, 15 joints
Links:
- link link1bar: geometry visual cylinder length=0.1 radius=0.01
- link link1sail: geometry visual box size=0.01 0.02 0.05
- link link2bar: geometry visual cylinder length=0.25 radius=0.01
- link link2sail: geometry visual box size=0.01 0.1 0.02
- link link3bar: geometry visual cylinder length=0.2 radius=0.01
- link link3sail: geometry visual box size=0.01 0.1 0.02
- link pitch1motor: geometry visual cylinder length=0.1 radius=0.02
- link pitch2motor: geometry visual cylinder length=0.1 radius=0.02
- link table: geometry visual box size=0.2 0.15 0.0127
- link tipball: geometry visual sphere radius=0.02
- link yawmotor: geometry visual cylinder length=0.02 radius=0.03
Joints:
- joint shifttotip: origin xyz=0 1 0 rpy=0 0 0 -> xyz=0 0.2 0 rpy=0 0 0
- joint theta1: origin xyz=0 0 0 rpy=0 0 0 -> xyz=0 0 0.1 rpy=0 0 0
- joint theta3: origin xyz=0 1 0 rpy=0 0 0 -> xyz=0 0.25 0 rpy=0 0 0

Commit message: Modify code to run HEBI robot
Create launch file for HEBI robot, change holding trajectory to quintic spline from initial to q_init, and modify urdf to be consistent with rotation direction of actual robot

File: urdf/threeDOF.urdf (robot description, URDF)
Before this commit: robot threeDOF, 16 links, 15 joints
Joints:
- joint theta3: axis 1 0 0 -> -1 0 0

Commit message: Update threeDOF.urdf
Update urdf with dimensions as measured from actual robot

File: urdf/threeDOF.urdf (robot description, URDF)
Before this commit: robot threeDOF, 16 links, 15 joints
Joints:
- joint theta1: origin xyz=0 0 0.1 rpy=0 0 0 -> xyz=0 0 0.085 rpy=0 0 0
