Commit message: Retriever URDF
retriever urdf

File: urdf/retriever.urdf (robot description, URDF)
Before this commit: robot retriever, 16 links, 15 joints
Links:
- removed link tipball
- added link pitch3motor; visual cylinder length=0.1 radius=0.02
- link link1bar: geometry visual cylinder length=0.0445 radius=0.01
- link link2bar: geometry visual cylinder length=0.4064 radius=0.01
- link link3bar: geometry visual cylinder length=0.4064 radius=0.01
- link pitch1motor: geometry visual cylinder length=0.045 radius=0.02
- link yawmotor: geometry visual cylinder length=0.03 radius=0.03
Joints:
- removed joint attach-tipball
- added joint attach-pitch3motor: type fixed, parent link3, child pitch3motor
- joint theta1: origin xyz=0 0 0.085 rpy=0 0 0 -> xyz=0 0 0.04 rpy=0 0 0
- joint theta3: origin xyz=0 0.25 0 rpy=0 0 0 -> xyz=0 0.4064 0 rpy=0 0 0
