Commit message: Gravity Compensation
Implemented gravity compensation, tuned the corresponding gravity parameters, and made some small changes to the urdf files.

File: urdf/ReceiveAssem.urdf (robot description, URDF)
Before this commit: robot ReceiveAssem, 7 links, 6 joints
Links:
- removed link Tip
- added link tip
Joints:
- joint Gripper: child Tip -> tip

File: urdf/ThrowerAssem.urdf (robot description, URDF)
Before this commit: robot ThrowerAssem, 5 links, 4 joints
Links:
- removed link Tip
- added link tip
Joints:
- removed joint Scoop
- added joint scoop: type fixed, parent Arm, child tip, origin xyz=0.0 -0.529 0.0454 rpy=0 0 0
- joint Tilt: child Arm -> tip

Commit message: fix receiver urdf
fix urdf for horizontal 0 position

File: urdf/ReceiveAssem.urdf (robot description, URDF)
Before this commit: robot ReceiveAssem, 7 links, 6 joints
Joints:
- joint Tilt: origin xyz=-0.0889 0 0.05135 rpy=0 -1.5707963267949 3.14159265358979 -> xyz=-0.0889 0 0.05135 rpy=1.5707963267949 0 1.5707963267949

Commit message: Converting from joint space to task space
debugged a lot and made progress in converting code to task space. ikin not converging and jacobian inverse method makes arm shoot forwards.

File: urdf/ReceiveAssem.urdf (robot description, URDF)
Before this commit: robot ReceiveAssem, 7 links, 6 joints
Joints:
- joint Wrist: type continuous -> fixed

Commit message: Thrower Test Update
Update Thrower Test with compute spline and callback event

File: urdf/ReceiveAssem.urdf (robot description, URDF)
Before this commit: robot ReceiveAssem, 7 links, 6 joints
Joints:
- joint Gripper: origin xyz=0 0.1 -0.0325 rpy=0 0 0 -> xyz=0 0.0 -0.0325 rpy=0 0 0
